File: HARDWARE/ETH16CDAQ1/Ethernet.kicad_sch (KiCad schematic)
At the start: 25 parts, among them J301 RJ45_Wuerth_7499010121A, U301 LAN8742A, Y301 NX5032GA-25

Commit message: Development
Parts:
- Y301: footprint ETH1ACPL-C79x:NX5032GA -> ETH16CDAQ1:NX5032GA
Changed lines of the file:
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@@
 			)
 		)
-		(property "Footprint" "ETH1ACPL-C79x:NX5032GA"
+		(property "Footprint" "ETH16CDAQ1:NX5032GA"
 			(at 80.01 125.73 0)
 			(effects

Commit message: Development
Changed lines of the file:
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@@
-	(wire
-		(pts
-			(xy 91.44 30.48) (xy 91.44 31.75)
-		)
-		(stroke
-			(width 0)
-			(type default)
-		)
-	)
 	(wire
 		(pts
@@
 					(unit 1)
 				)
-			)
-		)
-	)
-	(symbol
-		(lib_id "power:PWR_FLAG")
-		(at 91.44 30.48 0)
-		(unit 1)
-		(exclude_from_sim no)
-		(in_bom yes)
-		(on_board yes)
-		(dnp no)
-		(property "Reference" "#FLG0302"
-			(at 91.44 28.575 0)
-			(effects
-				(font
-					(size 1.27 1.27)
-				)
-				(hide yes)
-			)
-		)
-		(property "Value" "PWR_FLAG"
-			(at 91.44 26.162 0)
-			(effects
-				(font
-					(size 1.27 1.27)
-				)
-			)
-		)
-		(property "Footprint" ""
-			(at 91.44 30.48 0)
-			(effects
-				(font
-					(size 1.27 1.27)
-				)
-				(hide yes)
-			)
-		)
-		(property "Datasheet" "~"
-			(at 91.44 30.48 0)
-			(effects
-				(font
-					(size 1.27 1.27)
-				)
-				(hide yes)
-			)
-		)
-		(property "Description" "Special symbol for telling ERC where power comes from"
-			(at 91.44 30.48 0)
-			(effects
-				(font
-					(size 1.27 1.27)
-				)
-				(hide yes)
-			)
-		)
-		(pin "1"
-		)
-		(instances
-			(project "ETH16CDAQ1"
-				(path "/2ab14781-f8f9-43b8-b10b-375641815f01/fd2c9437-3b30-4ac8-a45b-dc5aa1d5f777"
-					(reference "#FLG0302")
-					(unit 1)
-				)
-			)
-			(project "ETH1HMSR-SMS"
-				(path "/c9f88626-4b87-4d35-a77a-42f8d5451fae/6cffac93-e144-4206-a1fa-eb6db2a641b5"
-					(reference "#FLG02")
-					(unit 1)
-				)
-			)
-			(project "ETH1ACPL-C79x"
-				(path "/e8a00664-7a76-490e-9471-410cd41c5487/2901751b-a680-4678-bb03-eb29728a9ca7"
-					(reference "#FLG0402")
-					(unit 1)
-				)

Commit message: Development
Changed lines of the file:
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@@
 		(fields_autoplaced yes)
 		(property "Reference" "RN302"
-			(at 101.6 168.275 0)
+			(at 101.6 167.6399 0)
 			(effects
 				(font
@@
 		)
 		(property "Value" "EXB-V8V103JV"
-			(at 101.6 170.815 0)
+			(at 101.6 170.1799 0)
 			(effects
 				(font
