File: HARDWARE/ETH16CDAQ1/ETH16CDAQ1.kicad_sch (KiCad schematic)
At the start: 0 parts

Commit message: Development
Parts:
- added H101, H102, H103, H104: MountingHole, MountingHole:MountingHole_3.2mm_M3_DIN965_Pad, symbol Mechanical:MountingHole
- added HS101: Heatsink, ETH16CDAQ1:960-19-12-S-AB-0, symbol Mechanical:Heatsink

Commit message: Development
Other:
- sheet MCU ports: added MUX1_A0, MUX1_A1, MUX1_A2, MUX2_A0, MUX2_A1, MUX2_A2, MUX_EN, OUT+, OUT-, SPI_MISO, SPI_MOSI, SPI_SCLK, SPI_~{CS}; removed none

Commit message: Development
Parts:
- H103, H104: footprint MountingHole:MountingHole_3.2mm_M3_DIN965_Pad -> MountingHole:MountingHole_2.2mm_M2_DIN965
Other:
- sheet Analog ports: added GND_CTR, RCTR[1..16]; removed MUX1_A0, MUX1_A1, MUX1_A2, MUX2_A0, MUX2_A1, MUX2_A2, MUX_EN
- sheet MCU ports: added GND_CTR, RCTR[1..16]; removed MUX1_A0, MUX1_A1, MUX1_A2, MUX2_A0, MUX2_A1, MUX2_A2, MUX_EN
- moved on the sheet: HS101
Changed lines of the file:
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@@
 	(generator_version "8.0")
 	(paper "A4")
+	(bus
+		(pts
+			(xy 119.38 62.23) (xy 124.46 62.23)
+		)
+		(stroke
+			(width 0)
+			(type default)
+		)
+	)
 	(wire
 		(pts
@@
 	(wire
 		(pts
-			(xy 119.38 74.93) (xy 124.46 74.93)
-		)
-		(stroke
-			(width 0)
-			(type default)
-		)
-	)
-	(wire
-		(pts
 			(xy 119.38 83.82) (xy 124.46 83.82)
 		)
@@
 	(wire
 		(pts
-			(xy 119.38 72.39) (xy 124.46 72.39)
-		)
-		(stroke
-			(width 0)
-			(type default)
-		)
-	)
-	(wire
-		(pts
 			(xy 119.38 55.88) (xy 124.46 55.88)
 		)
@@
 	(wire
 		(pts
-			(xy 119.38 62.23) (xy 124.46 62.23)
-		)
-		(stroke
-			(width 0)
-			(type default)
-		)
-	)
-	(wire
-		(pts
 			(xy 168.91 57.15) (xy 173.99 57.15)
 		)
@@
 	(wire
 		(pts
-			(xy 119.38 59.69) (xy 124.46 59.69)
-		)
-		(stroke
-			(width 0)
-			(type default)
-		)
-	)
-	(wire
-		(pts
 			(xy 119.38 53.34) (xy 124.46 53.34)
 		)
@@
 	(wire
 		(pts
-			(xy 119.38 69.85) (xy 124.46 69.85)
+			(xy 119.38 66.04) (xy 124.46 66.04)
 		)
 		(stroke
@@
 	(wire
 		(pts
-			(xy 119.38 64.77) (xy 124.46 64.77)
-		)
-		(stroke
-			(width 0)
-			(type default)
-		)
-	)
-	(wire
-		(pts
 			(xy 119.38 88.9) (xy 124.46 88.9)
-		)
-		(stroke
-			(width 0)
-			(type default)
-		)
-	)
-	(wire
-		(pts
-			(xy 119.38 67.31) (xy 124.46 67.31)
 		)
 		(stroke
@@
 			)
 		)
-		(property "Footprint" "MountingHole:MountingHole_3.2mm_M3_DIN965_Pad"
+		(property "Footprint" "MountingHole:MountingHole_2.2mm_M2_DIN965"
 			(at 19.05 185.42 0)
 			(effects
@@
 			)
 		)
-		(property "Footprint" "MountingHole:MountingHole_3.2mm_M3_DIN965_Pad"
+		(property "Footprint" "MountingHole:MountingHole_2.2mm_M2_DIN965"
 			(at 19.05 191.77 0)
 			(effects
@@
 	(symbol
 		(lib_id "Mechanical:Heatsink")
-		(at 45.72 181.61 0)
+		(at 19.05 166.37 0)
 		(unit 1)
 		(exclude_from_sim yes)
@@
 		(fields_autoplaced yes)
 		(property "Reference" "HS101"
-			(at 49.53 178.4349 0)
+			(at 22.86 163.1949 0)
 			(effects
 				(font
@@
 		)
 		(property "Value" "Heatsink"
-			(at 49.53 180.9749 0)
+			(at 22.86 165.7349 0)
 			(effects
 				(font
@@
 		)
 		(property "Footprint" "ETH16CDAQ1:960-19-12-S-AB-0"
-			(at 46.0248 181.61 0)
+			(at 19.3548 166.37 0)
 			(effects
 				(font
@@
 		)
 		(property "Datasheet" "~"
-			(at 46.0248 181.61 0)
+			(at 19.3548 166.37 0)
 			(effects
 				(font
@@
 		)
 		(property "Description" "Heatsink"
-			(at 45.72 181.61 0)
+			(at 19.05 166.37 0)
 			(effects
 				(font
@@
 			)
 		)
-		(pin "MUX2_A2" input
-			(at 119.38 74.93 0)
-			(effects
-				(font
-					(size 1.27 1.27)
-				)
-				(justify right)
-			)
-		)
-		(pin "MUX2_A1" input
-			(at 119.38 72.39 0)
-			(effects
-				(font
-					(size 1.27 1.27)
-				)
-				(justify right)
-			)
-		)
-		(pin "MUX2_A0" input
-			(at 119.38 69.85 0)
-			(effects
-				(font
-					(size 1.27 1.27)
-				)
-				(justify right)
-			)
-		)
-		(pin "MUX_EN" input
-			(at 119.38 67.31 0)
-			(effects
-				(font
-					(size 1.27 1.27)
-				)
-				(justify right)
-			)
-		)
-		(pin "MUX1_A1" input
-			(at 119.38 62.23 0)
-			(effects
-				(font
-					(size 1.27 1.27)
-				)
-				(justify right)
-			)
-		)
-		(pin "MUX1_A2" input
-			(at 119.38 64.77 0)
-			(effects
-				(font
-					(size 1.27 1.27)
-				)
-				(justify right)
-			)
-		)
-		(pin "MUX1_A0" input
-			(at 119.38 59.69 0)
-			(effects
-				(font
-					(size 1.27 1.27)
-				)
-				(justify right)
-			)
-		)
 		(pin "OUT-" output
 			(at 119.38 55.88 0)
@@
 		(pin "SPI_MISO" output
 			(at 119.38 88.9 0)
+			(effects
+				(font
+					(size 1.27 1.27)
+				)
+				(justify right)
+			)
+		)
+		(pin "RCTR[1..16]" bidirectional
+			(at 119.38 62.23 0)
+			(effects
+				(font
+					(size 1.27 1.27)
+				)
+				(justify right)
+			)
+		)
+		(pin "GND_CTR" input
+			(at 119.38 66.04 0)
 			(effects
 				(font
@@
 			)
 		)
-		(pin "MUX1_A1" output
-			(at 124.46 62.23 180)
-			(effects
-				(font
-					(size 1.27 1.27)
-				)
-				(justify left)
-			)
-		)
-		(pin "MUX1_A0" output
-			(at 124.46 59.69 180)
-			(effects
-				(font
-					(size 1.27 1.27)
-				)
-				(justify left)
-			)
-		)
-		(pin "MUX_EN" output
-			(at 124.46 67.31 180)
-			(effects
-				(font
-					(size 1.27 1.27)
-				)
-				(justify left)
-			)
-		)
 		(pin "SPI_~{CS}" output
 			(at 124.46 81.28 180)
@@
 			)
 		)
-		(pin "MUX2_A2" output
-			(at 124.46 74.93 180)
-			(effects
-				(font
-					(size 1.27 1.27)
-				)
-				(justify left)
-			)
-		)
 		(pin "SPI_MISO" input
 			(at 124.46 88.9 180)
@@
 			)
 		)
-		(pin "MUX2_A1" output
-			(at 124.46 72.39 180)
-			(effects
-				(font
-					(size 1.27 1.27)
-				)
-				(justify left)
-			)
-		)
-		(pin "MUX2_A0" output
-			(at 124.46 69.85 180)
-			(effects
-				(font
-					(size 1.27 1.27)
-				)
-				(justify left)
-			)
-		)
-		(pin "MUX1_A2" output
-			(at 124.46 64.77 180)
-			(effects
-				(font
+		(pin "RCTR[1..16]" bidirectional
+			(at 124.46 62.23 180)
+			(effects
+				(font
+					(size 1.27 1.27)
+				)
+				(justify left)
+			)
+		)
+		(pin "GND_CTR" output
+			(at 124.46 66.04 180)
+			(effects
+				(font

Commit message: Development
Other:
- sheet Analog ports: added GND1_CTR, GND2_CTR; removed GND_CTR
- sheet MCU ports: added GND1_CTR, GND2_CTR; removed GND_CTR
Changed lines of the file:
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@@
+	(wire
+		(pts
+			(xy 119.38 68.58) (xy 124.46 68.58)
+		)
+		(stroke
+			(width 0)
+			(type default)
+		)
+	)
 	(wire
 		(pts
@@
 			)
 		)
-		(pin "GND_CTR" input
+		(pin "GND1_CTR" input
 			(at 119.38 66.04 0)
+			(effects
+				(font
+					(size 1.27 1.27)
+				)
+				(justify right)
+			)
+		)
+		(pin "GND2_CTR" input
+			(at 119.38 68.58 0)
 			(effects
 				(font
@@
 			)
 		)
-		(pin "GND_CTR" output
+		(pin "GND1_CTR" output
 			(at 124.46 66.04 180)
 			(effects
 				(font
+					(size 1.27 1.27)
+				)
+				(justify left)
+			)
+		)
+		(pin "GND2_CTR" output
+			(at 124.46 68.58 180)
+			(effects
+				(font

Commit message: Development
Parts:
- HS101: value Heatsink -> 960-19-12-S-AB-0
Changed lines of the file:
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@@
 			)
 		)
-		(property "Value" "Heatsink"
+		(property "Value" "960-19-12-S-AB-0"
 			(at 22.86 165.7349 0)
 			(effects
