File: HARDWARE/ETH16CDAQ1/ETH16CDAQ1.kicad_pcb (KiCad board)
At the start: 2 copper layers, 100 x 45 mm, 111 parts, among them J201 20021111-00010T4LF, J301 RJ45_Wuerth_7499010121A, J401 5499141-4, J501 1715721, Q501 SI5618A, Q502 MMBT3904, U201 REF1933AIDDCT, U202 STM32H743VITx, U203 24LC08B-E/MS, U301 LAN8742A, U401 ADG5408BRUZ, U402 ADG5408BRUZ, U403 ADA4254ARUZ, U501 PDME2-S24-D24-S, U502 PDME2-S24-S9-S, U503 TLE4476D, U504 TPS7A39, Y201 NX5032GA-16, Y301 NX5032GA-25

Commit message: Development
Parts:
- C211, C219, C302, C305, C308, C309, C310, C311, C312, C402, C404, C405, C406, C501, C502: moved to B.Cu
- moved C311 252.0 mm to (182.2, 87.5), turned to 90 degrees
- moved C312 249.0 mm to (179.7, 100.5), turned to -90 degrees
- moved C307 241.7 mm to (167.9, 100.5), turned to -90 degrees
- moved C309 241.2 mm to (172.0, 96.4), turned to -90 degrees
- moved C305 241.0 mm to (167.1, 95.1), turned to -90 degrees
- moved C302 240.8 mm to (167.1, 91.8), turned to 90 degrees
- moved C308 239.4 mm to (170.1, 90.6), turned to 90 degrees
- moved C310 237.2 mm to (167.9, 100.5), turned to -90 degrees
- moved C211 159.9 mm to (148.6, 85.7)
- moved C405 158.0 mm to (129.7, 111.8), turned to 180 degrees
- moved C406 157.9 mm to (129.7, 114.0), turned to 180 degrees
- moved C219 150.5 mm to (143.6, 97.9)
- moved C402 147.2 mm to (122.8, 92.3)
- moved C404 146.9 mm to (122.2, 98.6)
- moved R402 10.5 mm to (129.3, 106.3), turned to 0 degrees
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Connections:
- net /Analog/AIN_1P renamed /Analog/AIN_1
- J401 pad 10: /Analog/AIN_4N -> /Analog/AIN_8
- J401 pad 11: /Analog/AIN_5P -> /Analog/AIN_9
- J401 pad 12: /Analog/AIN_5N -> /Analog/AIN_10
- J401 pad 13: /Analog/AIN_6P -> /Analog/AIN_11
- J401 pad 14: /Analog/AIN_6N -> /Analog/AIN_12
- J401 pad 15: /Analog/AIN_7P -> /Analog/AIN_13
- J401 pad 16: /Analog/AIN_7N -> /Analog/AIN_14
- J401 pad 17: /Analog/AIN_8P -> /Analog/AIN_15
- J401 pad 18: /Analog/AIN_8N -> /Analog/AIN_16
- J401 pad 4: /Analog/AIN_1N -> /Analog/AIN_2
- J401 pad 5: /Analog/AIN_2P -> /Analog/AIN_3
- J401 pad 6: /Analog/AIN_2N -> /Analog/AIN_4
- J401 pad 7: /Analog/AIN_3P -> /Analog/AIN_5
- J401 pad 8: /Analog/AIN_3N -> /Analog/AIN_6
- J401 pad 9: /Analog/AIN_4P -> /Analog/AIN_7
- U202 pad 17: /MCU/OUT- -> /Analog/OUT-
- U202 pad 18: /MCU/OUT+ -> /Analog/OUT+
- U202 pad 34: unconnected-(U202-PB0-Pad34) -> /Analog/MUX2_A2
- U202 pad 35: unconnected-(U202-PB1-Pad35) -> /Analog/MUX2_A1
- U202 pad 36: unconnected-(U202-PB2-Pad36) -> /Analog/MUX2_A0
- U202 pad 37: unconnected-(U202-PE7-Pad37) -> /Analog/MUX_EN
- U202 pad 38: unconnected-(U202-PE8-Pad38) -> /Analog/MUX1_A0
- U202 pad 39: unconnected-(U202-PE9-Pad39) -> /Analog/MUX1_A1
- U202 pad 40: unconnected-(U202-PE10-Pad40) -> /Analog/MUX1_A2
- U202 pad 41: unconnected-(U202-PE11-Pad41) -> /Analog/SPI_~{CS}
- U202 pad 42: unconnected-(U202-PE12-Pad42) -> /Analog/SPI_SCLK
- U202 pad 43: unconnected-(U202-PE13-Pad43) -> /Analog/SPI_MISO
- U202 pad 44: unconnected-(U202-PE14-Pad44) -> /Analog/SPI_MOSI
- U202 pad 64: /MCU/LED_RED -> /MCU/LED_GREEN
- U202 pad 65: /MCU/LED_GREEN -> /MCU/LED_RED
- U401 pad 10: /Analog/AIN_7P -> /Analog/AIN_5
- U401 pad 11: /Analog/AIN_6P -> /Analog/AIN_8
- U401 pad 12: /Analog/AIN_5P -> /Analog/AIN_7
- U401 pad 5: /Analog/AIN_2P -> /Analog/AIN_2
- U401 pad 6: /Analog/AIN_3P -> /Analog/AIN_3
- U401 pad 7: /Analog/AIN_4P -> /Analog/AIN_4
- U401 pad 9: /Analog/AIN_8P -> /Analog/AIN_6
- U402 pad 10: /Analog/AIN_7N -> /Analog/AIN_13
- U402 pad 11: /Analog/AIN_6N -> /Analog/AIN_16
- U402 pad 12: /Analog/AIN_5N -> /Analog/AIN_15
- U402 pad 4: /Analog/AIN_1N -> /Analog/AIN_9
- U402 pad 5: /Analog/AIN_2N -> /Analog/AIN_10
- U402 pad 6: /Analog/AIN_3N -> /Analog/AIN_11
- U402 pad 7: /Analog/AIN_4N -> /Analog/AIN_12
- U402 pad 9: /Analog/AIN_8N -> /Analog/AIN_14
Routing:
- net +3.3V: track 0.00 -> 52.3 mm, vias 0 -> 16
- net /Analog/OUT-: track 0.00 -> 46.1 mm
- net +3.3VADC: track 0.00 -> 45.8 mm, vias 0 -> 2
- net /MCU/NRST: track 0.00 -> 44.6 mm, vias 0 -> 2
- net /Ethernet/RMII_MDIO: track 0.00 -> 44.4 mm, vias 0 -> 2
- net /Analog/OUT+: track 0.00 -> 44.3 mm
- net /Ethernet/REF_CLK: track 0.00 -> 39.1 mm, vias 0 -> 2
- net /Ethernet/RMII_TXD0: track 0.00 -> 39.1 mm, vias 0 -> 2
- net /Ethernet/RMII_TXD1: track 0.00 -> 39.0 mm, vias 0 -> 2
- net /Ethernet/RMII_TXEN: track 0.00 -> 39.0 mm, vias 0 -> 2
- net /Ethernet/RMII_MDC: track 0.00 -> 39.0 mm, vias 0 -> 2
- net /Ethernet/RMII_CRS_DV: track 0.00 -> 38.9 mm, vias 0 -> 2
- net /Ethernet/RMII_RXD1: track 0.00 -> 38.8 mm, vias 0 -> 2
- net /Ethernet/RMII_RXD0: track 0.00 -> 38.6 mm, vias 0 -> 2
- net /Analog/MUX_EN: track 0.00 -> 36.7 mm, vias 0 -> 3
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- added copper zone on B.Cu, net +3.3V
- added copper zone on F.Cu, net +3.3V
- added copper zone on In2.Cu, net +3.3V
- added copper zone on B.Cu, net +5V
- added copper zone on F.Cu, net +5V
- added copper zone on In2.Cu, net +5V
- added copper zone on B.Cu, net GND
- added copper zone on F.Cu, net GND
- added copper zone on In1.Cu, net GND
- added copper zone on B.Cu, net GNDPWR
- added copper zone on In1.Cu, net GNDPWR
- added copper zone on B.Cu, net Net-(D501-K)
- added copper zone on F.Cu, net Net-(D501-K)
- added copper zone on In2.Cu, net Net-(D501-K)
- added copper zone on F.Cu, net Net-(D502-K)
- added copper zone on B.Cu, net Net-(J501-Pin_1)
- added copper zone on B.Cu, net Net-(Q501-D)
- added copper zone on F.Cu, net Net-(Q501-D)
- added copper zone on B.Cu, net Net-(U501-+Vin)
- added copper zone on F.Cu, net Net-(U501-+Vin)
- added copper zone on In2.Cu, net Net-(U501-+Vin)
- added copper zone on B.Cu, net Net-(U501-+Vout)
- added copper zone on F.Cu, net Net-(U501-+Vout)
- added copper zone on B.Cu, net Net-(U501--Vout)
- added copper zone on F.Cu, net Net-(U501--Vout)
- added copper zone on B.Cu, net Net-(U502-+Vout)
- added copper zone on F.Cu, net Net-(U502-+Vout)
- added copper zone on F.Cu, net VPP
- added copper zone on In2.Cu, net VPP
- added copper zone on F.Cu, net VSS
- added copper zone on In2.Cu, net VSS
Other:
- copper layers 2 -> 4

Commit message: Development
Parts:
- removed the C401 at (122.8, 102.2)
- removed the C403 at (122.2, 108.7)
- removed the C405 at (129.7, 111.8)
- removed C406: 0.1u, Capacitor_SMD:C_0603_1608Metric_Pad1.08x0.95mm_HandSolder
- removed the U401 at (122.3, 105.5)
- removed U402: ADG5408BRUZ, Package_SO:TSSOP-16_4.4x5mm_P0.65mm
- added D401: 1N914WT, Diode_SMD:D_SOD-523, B.Cu at (112.0, 113.6)
- added D402: 1N914WT, Diode_SMD:D_SOD-523, B.Cu at (112.0, 112.2)
- added D403: 1N914WT, Diode_SMD:D_SOD-523, B.Cu at (112.0, 108.1)
- added D404: 1N914WT, Diode_SMD:D_SOD-523, B.Cu at (112.0, 104.0)
- added D405: 1N914WT, Diode_SMD:D_SOD-523, B.Cu at (112.0, 99.9)
- added D406: 1N914WT, Diode_SMD:D_SOD-523, B.Cu at (112.0, 95.8)
- added D407: 1N914WT, Diode_SMD:D_SOD-523, B.Cu at (112.0, 91.6)
- added D408: 1N914WT, Diode_SMD:D_SOD-523, B.Cu at (112.0, 87.5)
- added D409: 1N914WT, Diode_SMD:D_SOD-523, B.Cu at (120.4, 87.5)
- added D410: 1N914WT, Diode_SMD:D_SOD-523, B.Cu at (120.4, 91.6)
- added D411: 1N914WT, Diode_SMD:D_SOD-523, B.Cu at (120.4, 95.8)
- added D412: 1N914WT, Diode_SMD:D_SOD-523, B.Cu at (120.4, 99.9)
- added D413: 1N914WT, Diode_SMD:D_SOD-523, B.Cu at (120.4, 104.0)
- added D414: 1N914WT, Diode_SMD:D_SOD-523, B.Cu at (120.4, 108.1)
- added D415: 1N914WT, Diode_SMD:D_SOD-523, B.Cu at (120.4, 112.2)
- added D416: 1N914WT, Diode_SMD:D_SOD-523, B.Cu at (120.4, 116.3)
- added D417: 1N914WT, Diode_SMD:D_SOD-523, B.Cu at (120.4, 83.4)
- added K401: UMS05-1A80-75D, Relay_THT:Relay_StandexMeder_UMS, F.Cu at (111.3, 114.9)
- added K402: UMS05-1A80-75D, Relay_THT:Relay_StandexMeder_UMS, F.Cu at (111.3, 110.8)
- added K403: UMS05-1A80-75D, Relay_THT:Relay_StandexMeder_UMS, F.Cu at (111.3, 106.7)
- added K404: UMS05-1A80-75D, Relay_THT:Relay_StandexMeder_UMS, F.Cu at (111.3, 102.6)
- added K405: UMS05-1A80-75D, Relay_THT:Relay_StandexMeder_UMS, F.Cu at (111.3, 98.5)
- added K406: UMS05-1A80-75D, Relay_THT:Relay_StandexMeder_UMS, F.Cu at (111.3, 94.3)
- added K407: UMS05-1A80-75D, Relay_THT:Relay_StandexMeder_UMS, F.Cu at (111.3, 90.2)
- added K408: UMS05-1A80-75D, Relay_THT:Relay_StandexMeder_UMS, F.Cu at (111.3, 86.1)
- added K409: UMS05-1A80-75D, Relay_THT:Relay_StandexMeder_UMS, F.Cu at (119.6, 86.1)
- added K410: UMS05-1A80-75D, Relay_THT:Relay_StandexMeder_UMS, F.Cu at (119.6, 90.2)
- added K411: UMS05-1A80-75D, Relay_THT:Relay_StandexMeder_UMS, F.Cu at (119.6, 94.3)
- added K412: UMS05-1A80-75D, Relay_THT:Relay_StandexMeder_UMS, F.Cu at (119.6, 98.5)
- added K413: UMS05-1A80-75D, Relay_THT:Relay_StandexMeder_UMS, F.Cu at (119.6, 102.6)
- added K414: UMS05-1A80-75D, Relay_THT:Relay_StandexMeder_UMS, F.Cu at (119.6, 106.7)
- added K415: UMS05-1A80-75D, Relay_THT:Relay_StandexMeder_UMS, F.Cu at (119.6, 110.8)
- added K416: UMS05-1A80-75D, Relay_THT:Relay_StandexMeder_UMS, F.Cu at (119.6, 114.9)
- added K417: UMS05-1A80-75D, Relay_THT:Relay_StandexMeder_UMS, F.Cu at (119.6, 82.0)
- added Q401: BC817W, Package_TO_SOT_SMD:SOT-323_SC-70, B.Cu at (118.6, 119.8)
- added Q402: BC817W, Package_TO_SOT_SMD:SOT-323_SC-70, B.Cu at (115.8, 112.8)
- added Q403: BC817W, Package_TO_SOT_SMD:SOT-323_SC-70, B.Cu at (115.8, 108.7)
- added Q404: BC817W, Package_TO_SOT_SMD:SOT-323_SC-70, B.Cu at (115.8, 104.5)
- added Q405: BC817W, Package_TO_SOT_SMD:SOT-323_SC-70, B.Cu at (115.8, 100.5)
- added Q406: BC817W, Package_TO_SOT_SMD:SOT-323_SC-70, B.Cu at (115.8, 96.4)
- added Q407: BC817W, Package_TO_SOT_SMD:SOT-323_SC-70, B.Cu at (115.8, 92.2)
- added Q408: BC817W, Package_TO_SOT_SMD:SOT-323_SC-70, B.Cu at (115.8, 88.1)
- added Q409: BC817W, Package_TO_SOT_SMD:SOT-323_SC-70, B.Cu at (124.2, 88.3)
- added Q410: BC817W, Package_TO_SOT_SMD:SOT-323_SC-70, B.Cu at (124.2, 92.2)
- added Q411: BC817W, Package_TO_SOT_SMD:SOT-323_SC-70, B.Cu at (124.2, 96.4)
- added Q412: BC817W, Package_TO_SOT_SMD:SOT-323_SC-70, B.Cu at (124.2, 100.5)
- added Q413: BC817W, Package_TO_SOT_SMD:SOT-323_SC-70, B.Cu at (124.2, 104.5)
- added Q414: BC817W, Package_TO_SOT_SMD:SOT-323_SC-70, B.Cu at (124.2, 108.7)
- added Q415: BC817W, Package_TO_SOT_SMD:SOT-323_SC-70, B.Cu at (124.2, 112.8)
- added Q416: BC817W, Package_TO_SOT_SMD:SOT-323_SC-70, B.Cu at (124.2, 117.0)
- added Q417: BC817W, Package_TO_SOT_SMD:SOT-323_SC-70, B.Cu at (124.2, 84.1)
- added R401: 100k/0.1%, Resistor_SMD:R_0805_2012Metric_Pad1.20x1.40mm_HandSolder, B.Cu at (134.4, 109.6)
- added R402: 100k/0.1%, Resistor_SMD:R_0805_2012Metric_Pad1.20x1.40mm_HandSolder, B.Cu at (134.4, 114.8)
- added R403: 100k/0.1%, Resistor_SMD:R_0805_2012Metric_Pad1.20x1.40mm_HandSolder, B.Cu at (134.4, 111.6)
- added R404: 100k/0.1%, Resistor_SMD:R_0805_2012Metric_Pad1.20x1.40mm_HandSolder, B.Cu at (134.4, 116.8)
- added R407: 10k, Resistor_SMD:R_0603_1608Metric_Pad0.98x0.95mm_HandSolder, B.Cu at (127.4, 84.7)
- added RN202: EXB-V8V102JV, Resistor_SMD:R_Array_Concave_4x0603, B.Cu at (127.8, 114.9)
- added RN203: EXB-V8V102JV, Resistor_SMD:R_Array_Concave_4x0603, B.Cu at (127.8, 105.5)
- added RN204: EXB-V8V102JV, Resistor_SMD:R_Array_Concave_4x0603, B.Cu at (127.8, 94.6)
- added RN205: EXB-V8V102JV, Resistor_SMD:R_Array_Concave_4x0603, B.Cu at (127.8, 90.3)
- added RN401: MPMT1002AT1, Package_TO_SOT_SMD:SOT-23, F.Cu at (134.4, 110.4)
- added RN402: MPMT1002AT1, Package_TO_SOT_SMD:SOT-23, F.Cu at (134.4, 115.8)
- H103, H104: footprint MountingHole:MountingHole_3.2mm_M3_DIN965_Pad -> MountingHole:MountingHole_2.2mm_M2_DIN965
- U503: value TLE4476D -> TLE4476DXT
- moved C401 26.4 mm to (138.6, 113.5), turned to 180 degrees
- moved C402 23.8 mm to (138.6, 115.8), turned to 180 degrees
- moved C403 9.07 mm to (141.1, 117.5)
- moved C405 9.07 mm to (141.5, 108.1)
- moved R405 9.07 mm to (144.8, 108.1)
- moved U401 9.07 mm to (141.5, 113.5)
- moved C404 9.07 mm to (138.6, 110.9)
- moved R406 9.07 mm to (138.2, 108.1)
- moved H103 7.50 mm to (113.5, 81.5)
- moved H104 7.50 mm to (113.5, 119.5)
- moved J401 6.37 mm to (106.7, 111.9)
- moved C309 5.10 mm to (176.8, 94.7)
- moved C220 3.73 mm to (133.1, 88.6), turned to 90 degrees
- moved C221 3.64 mm to (134.6, 88.6), turned to 90 degrees
- moved C219 2.41 mm to (146.1, 97.9), turned to 180 degrees
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- renumbered C402 to C401, C404 to C402, C407 to C403, C408 to C404, C409 to C405, R401 to R405, R402 to R406, U403 to U401
Connections:
- J401 pad 1: GND -> GND3
- J401 pad 19: GND -> GND3
- J401 pad 2: GND -> GND3
- J401 pad 20: GND -> GND3
- U202 pad 25: unconnected-(U202-PA3-Pad25) -> /Analog/GND_CTR
- U202 pad 28: unconnected-(U202-PA4-Pad28) -> /MCU/RELAY15
- U202 pad 29: unconnected-(U202-PA5-Pad29) -> /MCU/RELAY16
- U202 pad 30: unconnected-(U202-PA6-Pad30) -> /MCU/RELAY14
- U202 pad 34: /Analog/MUX2_A2 -> /MCU/RELAY13
- U202 pad 35: /Analog/MUX2_A1 -> /MCU/RELAY12
- U202 pad 36: /Analog/MUX2_A0 -> /MCU/RELAY11
- U202 pad 37: /Analog/MUX_EN -> /MCU/RELAY10
- U202 pad 38: /Analog/MUX1_A0 -> /MCU/RELAY9
- U202 pad 39: /Analog/MUX1_A1 -> /MCU/RELAY8
- U202 pad 40: /Analog/MUX1_A2 -> /MCU/RELAY7
- U202 pad 45: unconnected-(U202-PE15-Pad45) -> /MCU/RELAY6
- U202 pad 46: unconnected-(U202-PB10-Pad46) -> /MCU/RELAY5
- U202 pad 54: unconnected-(U202-PB15-Pad54) -> /MCU/RELAY3
- U202 pad 55: unconnected-(U202-PD8-Pad55) -> /MCU/RELAY4
- U202 pad 56: unconnected-(U202-PD9-Pad56) -> /MCU/RELAY2
- U202 pad 57: unconnected-(U202-PD10-Pad57) -> /MCU/RELAY1
Routing:
- net GND: track 24.2 -> 189.2 mm, vias 13 -> 24
- net GND3: track 0.00 -> 52.9 mm
- net /Analog/D+: track 0.00 -> 50.5 mm, vias 0 -> 1
- net /Analog/D-: track 0.00 -> 38.9 mm, vias 0 -> 1
- net /Analog/MUX_EN: track 36.7 -> 0.00 mm, vias 3 -> 0
- net VSS: track 7.09 -> 43.7 mm, vias 6 -> 4
- net /Analog/MUX1_A0: track 31.6 -> 0.00 mm, vias 2 -> 0
- net VCCQ: track 15.4 -> 46.7 mm, vias 2 -> 5
- net /Analog/MUX1_A1: track 28.2 -> 0.00 mm, vias 2 -> 0
- net /MCU/RELAY1: track 0.00 -> 27.6 mm, vias 0 -> 1
- net /Analog/MUX1_A2: track 26.2 -> 0.00 mm, vias 2 -> 0
- net /MCU/RELAY2: track 0.00 -> 25.6 mm, vias 0 -> 1
- net /MCU/RELAY4: track 0.00 -> 25.5 mm, vias 0 -> 1
- net +5V: track 8.04 -> 32.6 mm
- net /MCU/RELAY3: track 0.00 -> 23.3 mm, vias 0 -> 1
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- added copper zone on B.Cu, net Earth
- added copper zone on F.Cu, net Earth
- added copper zone on B.Cu, net VCCQ
- added copper zone on F.Cu, net VCCQ
- added copper zone on In2.Cu, net VCCQ
- added copper zone on B.Cu, net VDDA
- added copper zone on B.Cu, net VPP
- added copper zone on B.Cu, net VSS

Commit message: Development
Parts:
- added D418: 1N914WT, Diode_SMD:D_SOD-523, B.Cu at (120.4, 120.5)
- added K418: UMS05-1A80-75D, Relay_THT:Relay_StandexMeder_UMS, F.Cu at (119.7, 119.0)
- added Q418: BC817W, Package_TO_SOT_SMD:SOT-323_SC-70, B.Cu at (124.2, 121.2)
- added R408: 10k, Resistor_SMD:R_0603_1608Metric_Pad0.98x0.95mm_HandSolder, B.Cu at (127.9, 120.5)
- moved Q401 9.27 mm to (109.6, 117.6), turned to 90 degrees
Connections:
- net /Analog/GND_CTR renamed /Analog/GND1_CTR
- net /Analog/RLY_GND renamed /Analog/RLY_GND1
- J401 pad 1: GND3 -> GND2
- J401 pad 19: GND3 -> GND1
- J401 pad 2: GND3 -> GND2
- J401 pad 20: GND3 -> GND1
- K417 pad 3: GND3 -> GND1
- U202 pad 58: unconnected-(U202-PD11-Pad58) -> /MCU/LED_BLUE
- U202 pad 59: unconnected-(U202-PD12-Pad59) -> /MCU/LED_GREEN
- U202 pad 60: unconnected-(U202-PD13-Pad60) -> /MCU/LED_RED
- U202 pad 63: /MCU/LED_BLUE -> /Analog/GND2_CTR
- U202 pad 64: /MCU/LED_GREEN -> unconnected-(U202-PC7-Pad64)
- U202 pad 65: /MCU/LED_RED -> unconnected-(U202-PC8-Pad65)
Routing:
- net GND3: track 52.9 -> 0.00 mm
- net /Analog/GND2_CTR: track 0.00 -> 35.2 mm, vias 0 -> 1
- net GND2: track 0.00 -> 23.8 mm
- net GND1: track 0.00 -> 23.5 mm
- net /Analog/RCTR2: track 12.0 -> 19.2 mm
- net GND: track 189.2 -> 194.7 mm, vias 24 -> 26
- net /Analog/RLY_2: track 10.4 -> 5.24 mm
- net /Analog/RLY_GND2: track 0.00 -> 3.89 mm
- net /Analog/OUT-: track 55.5 -> 52.9 mm
- net /Analog/OUT+: track 53.7 -> 51.1 mm
- net /MCU/LED_RED: track 22.5 -> 20.0 mm
- net /MCU/LED_BLUE: track 20.3 -> 17.9 mm
- net /MCU/LED_GREEN: track 20.7 -> 18.2 mm
- net Net-(Q418-B): track 0.00 -> 1.78 mm
- net +5V: track 32.6 -> 34.0 mm
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
Commit message: Development
Parts:
- removed C502: 4u7/50V, Capacitor_SMD:C_1206_3216Metric_Pad1.33x1.80mm_HandSolder
- removed C503, C504: 270p/2kV, Capacitor_SMD:C_1206_3216Metric_Pad1.33x1.80mm_HandSolder
- removed C513: 10u/25V, Capacitor_SMD:C_1206_3216Metric_Pad1.33x1.80mm_HandSolder
- removed U503: TLE4476DXT, Package_TO_SOT_SMD:TO-252-4
- added U505: RKZE-2405S, ETH16CDAQ1:CONV_RKZE-2405S, F.Cu at (171.2, 108.7)
- C403: moved to F.Cu
- C501: value 4u7/50V -> 10u/50V
- C507: value 2u2/25V -> 4u7/25V
- D201: value ASCB-JTC2-0A308 -> ASMB-MTB1-0A3A2
- L501: value IHLP2020BZER6R8M51 -> RLS-126-R; footprint Inductor_SMD:L_Vishay_IHLP-2020 -> ETH16CDAQ1:IND_RLS-126-R
- R401, R402, R403, R404: value 100k/0.1% -> 1Meg/0.1%; moved to F.Cu
- RN401, RN402: moved to B.Cu
- U501: value PDME2-S24-D24-S -> LM1117MP-3.3; footprint ETH16CDAQ1:CONV_PDME2-S24-D24-S -> Package_TO_SOT_SMD:SOT-223-3_TabPin2
- U502: value PDME2-S24-S9-S -> RB-2424D; footprint ETH16CDAQ1:CONV_PDME2-S24-S9-S -> ETH16CDAQ1:CONV_RB-2424D
- moved U501 18.9 mm to (155.2, 107.2)
- moved U502 9.15 mm to (171.1, 117.2)
- moved C403 5.66 mm to (146.4, 115.6), turned to 90 degrees
- moved R401 3.09 mm to (133.3, 112.5)
- moved R403 2.16 mm to (133.3, 109.7)
- moved R404 1.55 mm to (133.5, 118.1)
- moved C507 1.55 mm to (166.2, 108.7)
- moved C508 1.54 mm to (166.2, 106.3)
- moved C512 1.45 mm to (152.0, 107.8), turned to -90 degrees
- moved RN402 1.20 mm to (133.7, 114.8)
- moved R402 1.02 mm to (133.5, 115.3)
- moved RN401 0.99 mm to (133.7, 111.1)
- moved C506 0.80 mm to (170.9, 115.2)
- moved C510 0.80 mm to (168.5, 115.2)
- moved H101 0.50 mm to (196.5, 81.5)
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Connections:
- C505 pad 1: Net-(U501-+Vout) -> Net-(U502-+Vout)
- C506 pad 2: Net-(U501--Vout) -> Net-(U502--Vout)
- C507 pad 1: Net-(U502-+Vout) -> +5V
- C508 pad 1: Net-(U502-+Vout) -> +5V
- C509 pad 1: Net-(U501-+Vout) -> Net-(U502-+Vout)
- C510 pad 2: Net-(U501--Vout) -> Net-(U502--Vout)
- C512 pad 1: +5V -> +3.3V
- L501 pad 2: Net-(U501-+Vin) -> Net-(U502-+Vin)
- U501 pad 1: Net-(U501-+Vin) -> GND
- U501 pad 2: GNDPWR -> +3.3V
- U502 pad 1: Net-(U501-+Vin) -> Net-(U502-+Vin)
- U502 pad 4: GND -> Net-(U502--Vout)
- U504 pad 1: Net-(U501-+Vout) -> Net-(U502-+Vout)
- U504 pad 2: Net-(U501-+Vout) -> Net-(U502-+Vout)
- U504 pad 5: Net-(U501--Vout) -> Net-(U502--Vout)
Routing:
- net GND: track 194.7 -> 182.3 mm, vias 26 -> 32
- net Net-(U502-+Vout): track 11.8 -> 0.00 mm, vias 9 -> 0
- net +3.3V: track 51.4 -> 61.3 mm, vias 19 -> 20
- net +5V: track 34.0 -> 30.9 mm, vias 5 -> 1
- net Net-(U401-IN1+): track 12.8 -> 10.4 mm
- net Net-(U401-IN1-): track 9.40 -> 11.6 mm
- net /Analog/D+: track 50.5 -> 48.4 mm
- net Net-(U501-+Vin): track 1.64 -> 0.00 mm, vias 3 -> 0
- net GND2: track 23.8 -> 23.0 mm
- net /MCU/LED_GREEN: track 18.2 -> 17.6 mm
- net GND1: track 23.5 -> 22.9 mm
- added copper zone on F.Cu, net Net-(U502-+Vin)
- added copper zone on B.Cu, net Net-(U502--Vout)
- added copper zone on F.Cu, net Net-(U502--Vout)
- removed copper zone on B.Cu, net Net-(U501-+Vin)
- removed copper zone on F.Cu, net Net-(U501-+Vin)
- removed copper zone on In2.Cu, net Net-(U501-+Vin)
- removed copper zone on B.Cu, net Net-(U501-+Vout)
- removed copper zone on F.Cu, net Net-(U501-+Vout)
- removed copper zone on B.Cu, net Net-(U501--Vout)
- removed copper zone on F.Cu, net Net-(U501--Vout)
Other:
- board text added: "+24 VDC"
- board text added: "A1"
- board text added: "A10"
- board text added: "A11"
- board text added: "A12"
- board text added: "A13"
- board text added: "A14"
- board text added: "A15"
- board text added: "A16"
- board text added: "A2"
- board text added: "A3"
- board text added: "A4"
- board text added: "A5"
- board text added: "A6"
- board text added: "A7"
- board text added: "A8"
- board text added: "A9"
- board text added: "ETH16CDAQ1 V1.00 Default IP : 192.168.1.19"
- board text added: "GND1"
- board text added: "GND2"
- board text added: "M2"
- board text added: "VOLTAGE MEASUREMENT"

Commit message: Development
Parts:
- added C510: 10n, Capacitor_SMD:C_0603_1608Metric_Pad1.08x0.95mm_HandSolder, B.Cu at (152.5, 118.7)
- added C511: 10n, Capacitor_SMD:C_0603_1608Metric_Pad1.08x0.95mm_HandSolder, B.Cu at (151.5, 112.8)
- C502: renamed from C505; value 0.47u/50V -> 4u7/50V
- C503: renamed from C506; value 0.47u/50V -> 4u7/50V
- D201: value ASMB-MTB1-0A3A2 -> ASMB-MTB1-0B3A2
- HS101: value Heatsink -> 960-19-12-S-AB-0
- R503: value 167k -> 176k
- R506: value 176k -> 184k
- RN201: value 680 -> EXB-V8V102JV
- RN202, RN203, RN204, RN205: value EXB-V8V102JV -> EXB-V8V103JV
- moved C507 0.13 mm to (168.7, 115.2)
- moved C503 0.13 mm to (171.1, 115.2)
- renumbered C507 to C504, C508 to C505, C509 to C506, C510 to C507, C511 to C508, C512 to C509, C514 to C512, C515 to C513, U502 to U501, U505 to U502, U501 to U503
Routing:
- net VSS: track 43.3 -> 45.2 mm
- net VPP: track 23.3 -> 25.0 mm
- net Net-(U504-FBN): track 6.75 -> 7.59 mm, vias 0 -> 1
- net GND: track 182.3 -> 181.7 mm, vias 32 -> 31
- net /MCU/NRST: track 43.3 -> 43.9 mm
- net Net-(U504-FBP): track 5.98 -> 6.29 mm, vias 0 -> 1
