File: HARDWARE/ETH16CDAQ1/MCU.kicad_sch (KiCad schematic)
At the start: 34 parts, among them J201 20021111-00010T4LF, U201 REF1933AIDDCT, U202 STM32H743VITx, U203 24LC08B-E/MS, Y201 NX5032GA-16

Commit message: Development
Parts:
- Y201: footprint ETH1ACPL-C79x:NX5032GA -> ETH16CDAQ1:NX5032GA
Changed lines of the file:
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@@
 			)
 		)
-		(property "Footprint" "ETH1ACPL-C79x:NX5032GA"
+		(property "Footprint" "ETH16CDAQ1:NX5032GA"
 			(at 114.3 49.53 0)
 			(effects

Commit message: Development
Parts:
- U201: symbol ETH1ACPL-C79x:REF1933AIDDCT -> ETH16CDAQ1:REF1933AIDDCT
Connections:
- net LED_GREEN: now also U202.64 (PC7); no longer U202.65 (PC8)
- net LED_RED: no longer U202.64 (PC7)
- net MUX2_A2: now reaches U202.34 (PB0)
- net MUX2_A1: now reaches U202.35 (PB1)
- net MUX2_A0: now reaches U202.36 (PB2)
- net MUX_EN: now reaches U202.37 (PE7)
- net MUX1_A0: now reaches U202.38 (PE8)
- net MUX1_A1: now reaches U202.39 (PE9)
- net MUX1_A2: now reaches U202.40 (PE10)
- net SPI_~{CS}: now reaches U202.41 (PE11)
- net SPI_SCLK: now reaches U202.42 (PE12)
- net SPI_MISO: now reaches U202.43 (PE13)
- net SPI_MOSI: now reaches U202.44 (PE14)
- no-connect marks 66 -> 55
Changed lines of the file:
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@@
 	)
 	(no_connect
-		(at 187.96 74.93)
-	)
-	(no_connect
 		(at 144.78 102.87)
 	)
@@
 	)
 	(no_connect
-		(at 144.78 69.85)
-	)
-	(no_connect
 		(at 246.38 152.4)
 	)
@@
 	)
 	(no_connect
-		(at 144.78 77.47)
-	)
-	(no_connect
 		(at 144.78 118.11)
 	)
@@
 	)
 	(no_connect
-		(at 144.78 87.63)
-	)
-	(no_connect
 		(at 187.96 39.37)
 	)
 	(no_connect
-		(at 144.78 80.01)
-	)
-	(no_connect
 		(at 187.96 80.01)
 	)
@@
 	)
 	(no_connect
-		(at 144.78 72.39)
-	)
-	(no_connect
 		(at 187.96 151.13)
 	)
 	(no_connect
-		(at 144.78 82.55)
-	)
-	(no_connect
 		(at 246.38 149.86)
 	)
 	(no_connect
-		(at 187.96 77.47)
-	)
-	(no_connect
 		(at 187.96 29.21)
 	)
 	(no_connect
-		(at 144.78 85.09)
-	)
-	(no_connect
 		(at 30.48 31.75)
 	)
@@
 	)
 	(no_connect
-		(at 187.96 72.39)
-	)
-	(no_connect
 		(at 187.96 95.25)
 	)
@@
 	)
 	(no_connect
-		(at 144.78 74.93)
-	)
-	(no_connect
 		(at 187.96 97.79)
 	)
@@
 	(wire
 		(pts
+			(xy 143.51 69.85) (xy 144.78 69.85)
+		)
+		(stroke
+			(width 0)
+			(type default)
+		)
+	)
+	(wire
+		(pts
 			(xy 60.96 99.06) (xy 60.96 100.33)
 		)
@@
 	(wire
 		(pts
+			(xy 143.51 77.47) (xy 144.78 77.47)
+		)
+		(stroke
+			(width 0)
+			(type default)
+		)
+	)
+	(wire
+		(pts
 			(xy 187.96 118.11) (xy 189.23 118.11)
 		)
@@
 	(wire
 		(pts
+			(xy 187.96 74.93) (xy 189.23 74.93)
+		)
+		(stroke
+			(width 0)
+			(type default)
+		)
+	)
+	(wire
+		(pts
 			(xy 134.62 153.67) (xy 139.7 153.67)
 		)
@@
 	(wire
 		(pts
+			(xy 143.51 82.55) (xy 144.78 82.55)
+		)
+		(stroke
+			(width 0)
+			(type default)
+		)
+	)
+	(wire
+		(pts
 			(xy 22.86 41.91) (xy 22.86 53.34)
 		)
@@
 	(wire
 		(pts
+			(xy 143.51 74.93) (xy 144.78 74.93)
+		)
+		(stroke
+			(width 0)
+			(type default)
+		)
+	)
+	(wire
+		(pts
 			(xy 187.96 100.33) (xy 189.23 100.33)
 		)
@@
 	(wire
 		(pts
+			(xy 143.51 85.09) (xy 144.78 85.09)
+		)
+		(stroke
+			(width 0)
+			(type default)
+		)
+	)
+	(wire
+		(pts
 			(xy 110.49 181.61) (xy 116.84 181.61)
 		)
@@
 	(wire
 		(pts
+			(xy 187.96 77.47) (xy 189.23 77.47)
+		)
+		(stroke
+			(width 0)
+			(type default)
+		)
+	)
+	(wire
+		(pts
 			(xy 187.96 120.65) (xy 189.23 120.65)
 		)
@@
 	(wire
 		(pts
+			(xy 143.51 80.01) (xy 144.78 80.01)
+		)
+		(stroke
+			(width 0)
+			(type default)
+		)
+	)
+	(wire
+		(pts
 			(xy 246.38 154.94) (xy 257.81 154.94)
 		)
@@
 	(wire
 		(pts
+			(xy 143.51 87.63) (xy 144.78 87.63)
+		)
+		(stroke
+			(width 0)
+			(type default)
+		)
+	)
+	(wire
+		(pts
 			(xy 187.96 31.75) (xy 189.23 31.75)
 		)
@@
 	(wire
 		(pts
+			(xy 143.51 72.39) (xy 144.78 72.39)
+		)
+		(stroke
+			(width 0)
+			(type default)
+		)
+	)
+	(wire
+		(pts
 			(xy 25.4 41.91) (xy 25.4 53.34)
 		)
@@
 	(wire
 		(pts
+			(xy 187.96 72.39) (xy 189.23 72.39)
+		)
+		(stroke
+			(width 0)
+			(type default)
+		)
+	)
+	(wire
+		(pts
 			(xy 127 181.61) (xy 139.7 181.61)
 		)
@@
 	)
 	(label "LED_GREEN"
-		(at 212.09 135.89 180)
+		(at 212.09 133.35 180)
 		(fields_autoplaced yes)
 		(effects
@@
 	)
 	(label "LED_RED"
-		(at 212.09 133.35 180)
+		(at 214.63 139.7 180)
 		(fields_autoplaced yes)
 		(effects
@@
 		)
 	)
+	(hierarchical_label "MUX_EN"
+		(shape output)
+		(at 143.51 69.85 180)
+		(fields_autoplaced yes)
+		(effects
+			(font
+				(size 1.27 1.27)
+			)
+			(justify right)
+		)
+	)
+	(hierarchical_label "SPI_MISO"
+		(shape input)
+		(at 143.51 85.09 180)
+		(fields_autoplaced yes)
+		(effects
+			(font
+				(size 1.27 1.27)
+			)
+			(justify right)
+		)
+	)
+	(hierarchical_label "MUX2_A0"
+		(shape output)
+		(at 189.23 77.47 0)
+		(fields_autoplaced yes)
+		(effects
+			(font
+				(size 1.27 1.27)
+			)
+			(justify left)
+		)
+	)
 	(hierarchical_label "RMII_MDC"
 		(shape bidirectional)
@@
 		)
 	)
+	(hierarchical_label "MUX1_A1"
+		(shape output)
+		(at 143.51 74.93 180)
+		(fields_autoplaced yes)
+		(effects
+			(font
+				(size 1.27 1.27)
+			)
+			(justify right)
+		)
+	)
 	(hierarchical_label "RMII_TXD1"
 		(shape bidirectional)
@@
 		)
 	)
+	(hierarchical_label "MUX1_A0"
+		(shape output)
+		(at 143.51 72.39 180)
+		(fields_autoplaced yes)
+		(effects
+			(font
+				(size 1.27 1.27)
+			)
+			(justify right)
+		)
+	)
 	(hierarchical_label "REF_CLK"
 		(shape bidirectional)
@@
 		)
 	)
+	(hierarchical_label "SPI_MOSI"
+		(shape output)
+		(at 143.51 87.63 180)
+		(fields_autoplaced yes)
+		(effects
+			(font
+				(size 1.27 1.27)
+			)
+			(justify right)
+		)
+	)
+	(hierarchical_label "SPI_~{CS}"
+		(shape output)
+		(at 143.51 80.01 180)
+		(fields_autoplaced yes)
+		(effects
+			(font
+				(size 1.27 1.27)
+			)
+			(justify right)
+		)
+	)
+	(hierarchical_label "MUX2_A2"
+		(shape output)
+		(at 189.23 72.39 0)
+		(fields_autoplaced yes)
+		(effects
+			(font
+				(size 1.27 1.27)
+			)
+			(justify left)
+		)
+	)
 	(hierarchical_label "NRST"
 		(shape bidirectional)
@@
 		)
 	)
+	(hierarchical_label "MUX1_A2"
+		(shape output)
+		(at 143.51 77.47 180)
+		(fields_autoplaced yes)
+		(effects
+			(font
+				(size 1.27 1.27)
+			)
+			(justify right)
+		)
+	)
 	(hierarchical_label "OUT-"
 		(shape input)
@@
 		)
 	)
+	(hierarchical_label "MUX2_A1"
+		(shape output)
+		(at 189.23 74.93 0)
+		(fields_autoplaced yes)
+		(effects
+			(font
+				(size 1.27 1.27)
+			)
+			(justify left)
+		)
+	)
 	(hierarchical_label "RMII_RXD0"
 		(shape bidirectional)
@@
 		)
 	)
+	(hierarchical_label "SPI_SCLK"
+		(shape output)
+		(at 143.51 82.55 180)
+		(fields_autoplaced yes)
+		(effects
+			(font
+				(size 1.27 1.27)
+			)
+			(justify right)
+		)
+	)
 	(hierarchical_label "RMII_RXD1"
 		(shape bidirectional)
@@
 		(on_board yes)
 		(dnp no)
-		(fields_autoplaced yes)
 		(property "Reference" "#PWR0236"
 			(at 67.31 137.16 0)
@@
 		)
 		(property "Value" "VCOM"
-			(at 67.31 128.27 0)
+			(at 67.31 129.286 0)
 			(effects
 				(font
@@
 		(on_board yes)
 		(dnp no)
-		(fields_autoplaced yes)
 		(property "Reference" "#PWR0215"
 			(at 107.95 72.39 0)
@@
 	)
 	(symbol
-		(lib_id "ETH1ACPL-C79x:REF1933AIDDCT")
+		(lib_id "ETH16CDAQ1:REF1933AIDDCT")
 		(at 60.96 109.22 0)
 		(unit 1)

Commit message: Development
Parts:
- added RN202, RN203, RN204, RN205: EXB-V8V102JV, Resistor_SMD:R_Array_Concave_4x0603, symbol Device:R_Pack04
Connections:
- net LED_RED: now also U202.65 (PC8)
- net GND_CTR: now reaches U202.25 (PA3)
- net RELAY15: now reaches U202.28 (PA4)
- net RELAY15: now also RN205.5 (R4.2)
- net RELAY16: now reaches U202.29 (PA5)
- net RELAY16: now also RN205.6 (R3.2)
- net RELAY14: now reaches U202.30 (PA6)
- net RELAY14: now also RN205.7 (R2.2)
- net RELAY6: now reaches U202.45 (PE15)
- net RELAY6: now also RN203.7 (R2.2)
- net RELAY5: now reaches U202.46 (PB10)
- net RELAY5: now also RN203.8 (R1.2)
- net RELAY3: now reaches U202.54 (PB15)
- net RELAY3: now also RN202.5 (R4.2)
- net RELAY4: now reaches U202.55 (PD8)
- net RELAY4: now also RN202.6 (R3.2)
- net RELAY2: now reaches U202.56 (PD9)
- net RELAY2: now also RN202.7 (R2.2)
- net RELAY1: now reaches U202.57 (PD10)
- net RELAY1: now also RN202.8 (R1.2)
- net MUX1_A0 renamed RELAY9
- net RELAY9: now also RN204.8 (R1.2)
- net MUX1_A1 renamed RELAY8
- net RELAY8: now also RN203.5 (R4.2)
- net MUX1_A2 renamed RELAY7
- net RELAY7: now also RN203.6 (R3.2)
- net MUX2_A0 renamed RELAY11
- net RELAY11: now also RN204.6 (R3.2)
- net MUX2_A1 renamed RELAY12
- net RELAY12: now also RN204.5 (R4.2)
- net MUX2_A2 renamed RELAY13
- net RELAY13: now also RN205.8 (R1.2)
- net MUX_EN renamed RELAY10
- net RELAY10: now also RN204.7 (R2.2)
- new net RCTR1: RN202.1 (R1.1)
- new net RCTR10: RN204.2 (R2.1)
- new net RCTR11: RN204.3 (R3.1)
- new net RCTR12: RN204.4 (R4.1)
- new net RCTR13: RN205.1 (R1.1)
- new net RCTR14: RN205.2 (R2.1)
- new net RCTR15: RN205.4 (R4.1)
- new net RCTR16: RN205.3 (R3.1)
- new net RCTR2: RN202.2 (R2.1)
- new net RCTR3: RN202.4 (R4.1)
- new net RCTR4: RN202.3 (R3.1)
- new net RCTR5: RN203.1 (R1.1)
- new net RCTR6: RN203.2 (R2.1)
- new net RCTR7: RN203.3 (R3.1)
- new net RCTR8: RN203.4 (R4.1)
- new net RCTR9: RN204.1 (R1.1)
- no-connect marks 55 -> 45
Other:
- moved on the sheet: C202, C204, C205, C207, C220, C221, U201

Commit message: Development
Connections:
- net LED_BLUE: now also U202.58 (PD11); no longer U202.63 (PC6)
- net LED_GREEN: now also U202.59 (PD12); no longer U202.64 (PC7)
- net LED_RED: now also U202.60 (PD13); no longer U202.65 (PC8)
- net GND_CTR renamed GND1_CTR
- new net GND2_CTR: U202.63 (PC6)
- no-connect marks 45 -> 44
Changed lines of the file:
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@@
 	)
 	(no_connect
-		(at 246.38 152.4)
+		(at 187.96 135.89)
 	)
 	(no_connect
-		(at 187.96 107.95)
+		(at 246.38 152.4)
 	)
 	(no_connect
-		(at 144.78 125.73)
+		(at 187.96 107.95)
 	)
 	(no_connect
@@
 	)
 	(no_connect
-		(at 187.96 95.25)
+		(at 187.96 133.35)
 	)
 	(no_connect
-		(at 144.78 128.27)
+		(at 187.96 95.25)
 	)
 	(no_connect
@@
 	)
 	(no_connect
-		(at 144.78 123.19)
-	)
-	(no_connect
 		(at 233.68 152.4)
 	)
@@
 	(wire
 		(pts
-			(xy 187.96 133.35) (xy 212.09 133.35)
+			(xy 144.78 125.73) (xy 132.08 125.73)
 		)
 		(stroke
@@
 	(wire
 		(pts
-			(xy 187.96 135.89) (xy 212.09 135.89)
+			(xy 144.78 128.27) (xy 132.08 128.27)
 		)
 		(stroke
@@
 	(wire
 		(pts
+			(xy 187.96 130.81) (xy 189.23 130.81)
+		)
+		(stroke
+			(width 0)
+			(type default)
+		)
+	)
+	(wire
+		(pts
 			(xy 265.43 106.68) (xy 275.59 106.68)
 		)
@@
 	(wire
 		(pts
-			(xy 187.96 130.81) (xy 212.09 130.81)
+			(xy 144.78 123.19) (xy 132.08 123.19)
 		)
 		(stroke
@@
 	)
 	(label "LED_BLUE"
-		(at 212.09 130.81 180)
+		(at 132.08 123.19 0)
 		(fields_autoplaced yes)
 		(effects
@@
 				(size 1.27 1.27)
 			)
-			(justify right bottom)
+			(justify left bottom)
 		)
 	)
@@
 	)
 	(label "LED_GREEN"
-		(at 212.09 133.35 180)
+		(at 132.08 125.73 0)
 		(fields_autoplaced yes)
 		(effects
@@
 				(size 1.27 1.27)
 			)
-			(justify right bottom)
+			(justify left bottom)
 		)
 	)
@@
 	)
 	(label "LED_RED"
-		(at 212.09 135.89 180)
+		(at 132.08 128.27 0)
 		(fields_autoplaced yes)
 		(effects
@@
 				(size 1.27 1.27)
 			)
-			(justify right bottom)
+			(justify left bottom)
 		)
 	)
@@
 		)
 	)
+	(hierarchical_label "GND2_CTR"
+		(shape output)
+		(at 189.23 130.81 0)
+		(fields_autoplaced yes)
+		(effects
+			(font
+				(size 1.27 1.27)
+			)
+			(justify left)
+		)
+	)
 	(hierarchical_label "OUT-"
 		(shape input)
@@
 		)
 	)
-	(hierarchical_label "GND_CTR"
+	(hierarchical_label "GND1_CTR"
 		(shape output)
 		(at 189.23 36.83 0)

Commit message: Development
Parts:
- D201: value ASCB-JTC2-0A308 -> ASMB-MTB1-0B3A2
- RN201: value 680 -> EXB-V8V102JV
Changed lines of the file:
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@@
 	(wire
 		(pts
-			(xy 133.35 57.15) (xy 144.78 57.15)
+			(xy 134.62 57.15) (xy 144.78 57.15)
 		)
 		(stroke
@@
 	(wire
 		(pts
-			(xy 187.96 36.83) (xy 189.23 36.83)
+			(xy 187.96 36.83) (xy 201.93 36.83)
 		)
 		(stroke
@@
 	)
 	(label "MCU_DEF"
-		(at 133.35 57.15 0)
+		(at 134.62 57.15 0)
 		(fields_autoplaced yes)
 		(effects
@@
 	(hierarchical_label "GND1_CTR"
 		(shape output)
-		(at 189.23 36.83 0)
+		(at 201.93 36.83 0)
 		(fields_autoplaced yes)
 		(effects
@@
 		(on_board yes)
 		(dnp no)
-		(fields_autoplaced yes)
 		(property "Reference" "D201"
-			(at 46.99 22.86 90)
+			(at 47.244 23.368 90)
 			(effects
 				(font
@@
 			)
 		)
-		(property "Value" "ASCB-JTC2-0A308"
-			(at 54.61 25.4 90)
+		(property "Value" "ASMB-MTB1-0B3A2"
+			(at 54.61 25.908 90)
 			(effects
 				(font
@@
 		(fields_autoplaced yes)
 		(property "Reference" "RN201"
-			(at 33.02 35.56 0)
+			(at 33.02 35.5599 0)
 			(effects
 				(font
@@
 			)
 		)
-		(property "Value" "680"
-			(at 33.02 38.1 0)
+		(property "Value" "EXB-V8V102JV"
+			(at 33.02 38.0999 0)
 			(effects
 				(font
@@
 		(on_board yes)
 		(dnp no)
-		(fields_autoplaced yes)
 		(property "Reference" "U202"
-			(at 163.83 87.63 0)
+			(at 162.56 87.884 0)
 			(effects
 				(font
@@
 		)
 		(property "Value" "STM32H743VITx"
-			(at 157.48 94.615 0)
+			(at 157.734 94.488 0)
 			(effects
 				(font

Commit message: Development
Parts:
- RN202, RN203, RN204, RN205: value EXB-V8V102JV -> EXB-V8V103JV
Changed lines of the file:
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@@
 			)
 		)
-		(property "Value" "EXB-V8V102JV"
+		(property "Value" "EXB-V8V103JV"
 			(at 97.79 96.012 90)
 			(effects
@@
 			)
 		)
-		(property "Value" "EXB-V8V102JV"
+		(property "Value" "EXB-V8V103JV"
 			(at 97.79 112.268 90)
 			(effects
@@
 			)
 		)
-		(property "Value" "EXB-V8V102JV"
+		(property "Value" "EXB-V8V103JV"
 			(at 97.79 128.778 90)
 			(effects
@@
 			)
 		)
-		(property "Value" "EXB-V8V102JV"
+		(property "Value" "EXB-V8V103JV"
 			(at 97.79 79.502 90)
 			(effects
