File: HARDWARE/ETH16CDAQ1/Power.kicad_sch (KiCad schematic)
At the start: 35 parts, among them J501 1715721, Q501 SI5618A, Q502 MMBT3904, U501 PDME2-S24-D24-S, U502 TPS7A39, U503 PDME2-S24-S9-S, U504 TLE4476D

Commit message: Development
Parts:
- removed C511, C512: 4u7/50V, symbol Device:C
- removed L502: SRP3012CC-6R8M, symbol Device:L
- C501, C502, C503, C509, C510: footprint (none) -> Capacitor_SMD:C_1206_3216Metric_Pad1.33x1.80mm_HandSolder
- C504: renamed from C513; footprint (none) -> Capacitor_SMD:C_1206_3216Metric_Pad1.33x1.80mm_HandSolder
- C505: renamed from C504; footprint (none) -> Capacitor_SMD:C_1206_3216Metric_Pad1.33x1.80mm_HandSolder
- C506: renamed from C505; footprint (none) -> Capacitor_SMD:C_1206_3216Metric_Pad1.33x1.80mm_HandSolder
- C507: renamed from C514; footprint (none) -> Capacitor_SMD:C_1206_3216Metric_Pad1.33x1.80mm_HandSolder
- C508: renamed from C515; footprint (none) -> Capacitor_SMD:C_1206_3216Metric_Pad1.33x1.80mm_HandSolder
- C511: renamed from C506; footprint (none) -> Capacitor_SMD:C_0603_1608Metric_Pad1.08x0.95mm_HandSolder
- C512: renamed from C516; footprint (none) -> Capacitor_SMD:C_1206_3216Metric_Pad1.33x1.80mm_HandSolder
- C513: renamed from C517; footprint (none) -> Capacitor_SMD:C_1206_3216Metric_Pad1.33x1.80mm_HandSolder
- C514: renamed from C507; footprint (none) -> Capacitor_SMD:C_1206_3216Metric_Pad1.33x1.80mm_HandSolder
- C515: renamed from C508; footprint (none) -> Capacitor_SMD:C_1206_3216Metric_Pad1.33x1.80mm_HandSolder
- L501: value SRP3012CC-6R8M -> IHLP2020BZER6R8M51; footprint (none) -> Inductor_SMD:L_Vishay_IHLP-2020
- R503, R504, R505, R506: footprint (none) -> Resistor_SMD:R_0603_1608Metric_Pad0.98x0.95mm_HandSolder
- renumbered U503 to U502, U504 to U503, U502 to U504
Connections:
- net at C502.1, L501.2, U501.1 (+Vin): now also U502.1 (+Vin)
- net GNDPWR: now reaches C501.2, C502.2, C503.1, C504.1, J501.2 (Pin_2), R501.2, R502.2, U501.2 (-Vin), U502.2 (-Vin)
Other:
- moved on the sheet: C503, C504, C505, C506, C507, C508, C509, C510, C511, C512, C513, C514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

Commit message: Development
Parts:
- U503: value TLE4476D -> TLE4476DXT
Changed lines of the file:
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@@
 			)
 		)
-		(property "Value" "TLE4476D"
+		(property "Value" "TLE4476DXT"
 			(at 205.74 92.71 0)
 			(effects

Commit message: Development
Parts:
- removed C502: 4u7/50V, Capacitor_SMD:C_1206_3216Metric_Pad1.33x1.80mm_HandSolder, symbol Device:C
- removed C503, C504: 270p/2kV, Capacitor_SMD:C_1206_3216Metric_Pad1.33x1.80mm_HandSolder, symbol Device:C
- removed C513: 10u/25V, Capacitor_SMD:C_1206_3216Metric_Pad1.33x1.80mm_HandSolder, symbol Device:C
- removed U501: PDME2-S24-D24-S, ETH16CDAQ1:CONV_PDME2-S24-D24-S, symbol ETH16CDAQ1:PDME2-S24-D24-S
- removed U502: PDME2-S24-S9-S, ETH16CDAQ1:CONV_PDME2-S24-S9-S, symbol ETH16CDAQ1:PDME2-S24-S9-S
- removed U503: TLE4476DXT, Package_TO_SOT_SMD:TO-252-4, symbol ETH16CDAQ1:TLE4476D
- added U501: LM1117MP-3.3, Package_TO_SOT_SMD:SOT-223-3_TabPin2, symbol Regulator_Linear:LM1117MP-3.3
- added U502: RB-2424D, ETH16CDAQ1:CONV_RB-2424D, symbol ETH16CDAQ1:RB-2424D
- added U505: RKZE-2405S, ETH16CDAQ1:CONV_RKZE-2405S, symbol ETH16CDAQ1:RKZE-2405S
- C501: value 4u7/50V -> 10u/50V
- C507: value 2u2/25V -> 4u7/25V
- L501: value IHLP2020BZER6R8M51 -> RLS-126-R; footprint Inductor_SMD:L_Vishay_IHLP-2020 -> ETH16CDAQ1:IND_RLS-126-R
- R503: value 167k -> 176k
- R506: value 176k -> 184k
Connections:
- net +3.3V: now also C512.1, U501.2 (VO)
- net +5V: now also C507.1, C508.1, U501.3 (VI), U505.7 (+Vout); no longer C512.1
- net GND: now also U501.1 (GND), U502.5 (GND), U505.5 (-Vout)
- net GNDPWR: now also U502.2 (-Vin), U505.2 (-Vin)
- net at L501.2: now also U502.1 (+Vin), U505.1 (+Vin)
- net at C506.2, C510.2, U504.5 (INN): now also U502.4 (-Vout)
- net at C505.1, C509.1, U504.1 (INP)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: now also U502.6 (+Vout)
Other:
- moved on the sheet: C501, C512, D501, D502, F501, J501, L501, Q501, Q502, R501, R502

Commit message: Development
Parts:
- added C510, C511: 10n, Capacitor_SMD:C_0603_1608Metric_Pad1.08x0.95mm_HandSolder, symbol Device:C
- C502: renamed from C505; value 0.47u/50V -> 4u7/50V
- C503: renamed from C506; value 0.47u/50V -> 4u7/50V
- renumbered C507 to C504, C508 to C505, C509 to C506, C510 to C507, C511 to C508, C512 to C509, C514 to C512, C515 to C513, U502 to U501, U505 to U502, U501 to U503
Connections:
- net VPP: now also C510.1
- net VSS: now also C511.2
- net at R505.2, R506.1, U504.7 (FBN): now also C511.1
- net at R503.2, R504.1, U504.9 (FBP): now also C510.2
Other:
- moved on the sheet: C512, C513
